Commit message: Added IMU and sonar to the vehicle model, sensor frames added in URDF
Sonar is a gpu_lidar with 128x32 beams at 5 Hz, kept low since rendering
is on CPU. Server is now started with headless rendering.

File: src/auv_description/urdf/auv.urdf.xacro (robot description, xacro)
@@ -19,4 +19,29 @@
     </visual>
   </link>
+  <!-- sensor frames, poses are same as in auv_sim/models/auv/model.sdf.xacro -->
+  <link name="imu_link"/>
+  <joint name="imu_joint" type="fixed">
+    <parent link="base_link"/>
+    <child link="imu_link"/>
+    <origin xyz="0 0 0" rpy="0 0 0"/>
+  </joint>
+  <link name="dvl_link"/>
+  <joint name="dvl_joint" type="fixed">
+    <parent link="base_link"/>
+    <child link="dvl_link"/>
+    <origin xyz="0 0 -0.10" rpy="0 0 0"/>
+  </joint>
+  <link name="sonar_link">
+    <visual>
+      <origin xyz="0 0 0" rpy="0 1.5708 0"/>
+      <geometry><cylinder radius="0.03" length="0.06"/></geometry>
+      <material name="thruster_black"/>
+    </visual>
+  </link>
+  <joint name="sonar_joint" type="fixed">
+    <parent link="base_link"/>
+    <child link="sonar_link"/>
+    <origin xyz="0.22 0 -0.04" rpy="0 0.5236 0"/>
+  </joint>
   <xacro:macro name="thruster" params="name xyz rpy">
     <link name="${name}">

Commit message: Refactor AUV description: remove thruster configuration, update package description, and adjust RViz settings

File: src/auv_description/urdf/auv.urdf.xacro (robot description, xacro)
@@ -1,20 +1,16 @@
 <?xml version="1.0"?>
-<!-- Kinematic description for TF and RViz. Dynamics are in auv_sim/models/auv. -->
+<!--
+  Kinematic description of the torpedo AUV for TF and RViz. Dynamics are in
+  auv_sim/models/auv/model.sdf.xacro. Mesh is the MBARI Tethys LRAUV (Gazebo
+  Fuel, CC-BY 4.0), it is having the tail on +x, so it is turned by 180 deg to
+  get x forward as per REP-103.
+-->
 <robot name="auv" xmlns:xacro="http://www.ros.org/wiki/xacro">
-  <xacro:arg name="thrusters_file" default="$(find auv_description)/config/thrusters.yaml"/>
-  <xacro:property name="cfg" value="${xacro.load_yaml('$(arg thrusters_file)')}"/>
-  <material name="frame_blue"><color rgba="0.05 0.25 0.6 1.0"/></material>
-  <material name="foam_yellow"><color rgba="0.95 0.75 0.1 1.0"/></material>
-  <material name="thruster_black"><color rgba="0.1 0.1 0.1 1.0"/></material>
   <link name="base_link">
     <visual>
-      <origin xyz="0 0 -0.03" rpy="0 0 0"/>
-      <geometry><box size="0.44 0.30 0.12"/></geometry>
-      <material name="frame_blue"/>
-    </visual>
-    <visual>
-      <origin xyz="0 0 0.07" rpy="0 0 0"/>
-      <geometry><box size="0.44 0.34 0.07"/></geometry>
-      <material name="foam_yellow"/>
+      <origin xyz="0 0 0" rpy="0 0 3.14159265"/>
+      <geometry>
+        <mesh filename="package://auv_sim/models/auv/meshes/tethys.dae"/>
+      </geometry>
     </visual>
   </link>
@@ -32,38 +28,9 @@
     <origin xyz="0 0 -0.10" rpy="0 0 0"/>
   </joint>
-  <link name="sonar_link">
-    <visual>
-      <origin xyz="0 0 0" rpy="0 1.5708 0"/>
-      <geometry><cylinder radius="0.03" length="0.06"/></geometry>
-      <material name="thruster_black"/>
-    </visual>
-  </link>
+  <link name="sonar_link"/>
   <joint name="sonar_joint" type="fixed">
     <parent link="base_link"/>
     <child link="sonar_link"/>
-    <origin xyz="0.22 0 -0.04" rpy="0 0.5236 0"/>
+    <origin xyz="0.70 0 -0.08" rpy="0 0.5236 0"/>
   </joint>
-  <xacro:macro name="thruster" params="name xyz rpy">
-    <link name="${name}">
-      <visual>
-        <origin xyz="0 0 0" rpy="0 1.5708 0"/>
-        <geometry><cylinder radius="0.045" length="0.06"/></geometry>
-        <material name="thruster_black"/>
-      </visual>
-    </link>
-    <joint name="${name}_joint" type="fixed">
-      <parent link="base_link"/>
-      <child link="${name}"/>
-      <origin xyz="${xyz[0]} ${xyz[1]} ${xyz[2]}" rpy="${rpy[0]} ${rpy[1]} ${rpy[2]}"/>
-    </joint>
-  </xacro:macro>
-  <!-- xacro is not having a for loop, so going with recursion over the yaml list -->
-  <xacro:macro name="thruster_loop" params="i">
-    <xacro:if value="${i &lt; len(cfg['thrusters'])}">
-      <xacro:property name="t" value="${cfg['thrusters'][i]}"/>
-      <xacro:thruster name="${t['name']}" xyz="${t['xyz']}" rpy="${t['rpy']}"/>
-      <xacro:thruster_loop i="${i + 1}"/>
-    </xacro:if>
-  </xacro:macro>
-  <xacro:thruster_loop i="0"/>
 </robot>

Commit message: Added DVL beam sensor in vehicle model, DVL and GPS frames in URDF

File: src/auv_description/urdf/auv.urdf.xacro (robot description, xacro)
@@ -22,9 +22,23 @@
     <origin xyz="0 0 0" rpy="0 0 0"/>
   </joint>
+  <!-- DVL velocity is in dvl_link (body axes), beams are traced in dvl_beams_link (x down) -->
   <link name="dvl_link"/>
   <joint name="dvl_joint" type="fixed">
     <parent link="base_link"/>
     <child link="dvl_link"/>
-    <origin xyz="0 0 -0.10" rpy="0 0 0"/>
+    <origin xyz="0.3 0 -0.15" rpy="0 0 0"/>
+  </joint>
+  <link name="dvl_beams_link"/>
+  <joint name="dvl_beams_joint" type="fixed">
+    <parent link="base_link"/>
+    <child link="dvl_beams_link"/>
+    <origin xyz="0.3 0 -0.15" rpy="0 1.5708 0"/>
+  </joint>
+  <!-- GPS antenna on the top of the hull, out of water only at the surface -->
+  <link name="gps_link"/>
+  <joint name="gps_joint" type="fixed">
+    <parent link="base_link"/>
+    <child link="gps_link"/>
+    <origin xyz="-0.2 0 0.18" rpy="0 0 0"/>
   </joint>
   <link name="sonar_link"/>

Commit message: Added sonar fan sensor under the hull, forward sonar reduced to 64x16 for obstacle avoidance

File: src/auv_description/urdf/auv.urdf.xacro (robot description, xacro)
@@ -35,4 +35,11 @@
     <origin xyz="0.3 0 -0.15" rpy="0 1.5708 0"/>
   </joint>
+  <!-- across track sonar fan (multibeam and sidescan), x down -->
+  <link name="sonar_fan_link"/>
+  <joint name="sonar_fan_joint" type="fixed">
+    <parent link="base_link"/>
+    <child link="sonar_fan_link"/>
+    <origin xyz="0.1 0 -0.15" rpy="0 1.5708 0"/>
+  </joint>
   <!-- GPS antenna on the top of the hull, out of water only at the surface -->
   <link name="gps_link"/>

File: src/auv_sim/models/auv/model.sdf.xacro (robot description, xacro)
@@ -35,9 +35,13 @@
   <!-- DVL on the bottom of the hull, a bit ahead of the centre -->
   <xacro:property name="dvl_xyz" value="0.3 0 -0.15"/>
-  <!-- forward looking sonar on the nose, used for SLAM till the multibeam is added -->
+  <!-- across track acoustic fan under the hull, for the multibeam and the sidescan -->
+  <xacro:property name="fan_xyz" value="0.1 0 -0.15"/>
+  <xacro:property name="fan_samples" value="512"/>
+  <xacro:property name="fan_rate" value="10"/>
+  <!-- forward looking sonar on the nose, low resolution, for obstacle avoidance -->
   <xacro:property name="sonar_xyz" value="0.70 0 -0.08"/>
   <xacro:property name="sonar_pitch" value="0.5236"/>
-  <xacro:property name="sonar_h_samples" value="128"/>
-  <xacro:property name="sonar_v_samples" value="32"/>
+  <xacro:property name="sonar_h_samples" value="64"/>
+  <xacro:property name="sonar_v_samples" value="16"/>
   <xacro:property name="sonar_rate" value="5"/>
   <xacro:macro name="tethys_material">
@@ -203,4 +207,43 @@
       </sensor>
       <!--
+        Across track fan, 512 rays over +-85 deg from the nadir, in the plane
+        perpendicular to the hull. Sensor x is down and the horizontal sweep is
+        about the hull axis. The multibeam takes the inner +-60 deg of it and
+        the sidescan takes all of it (auv_sonar package).
+      -->
+      <sensor name="sonar_fan" type="gpu_lidar">
+        <pose>${fan_xyz} 0 ${pi / 2} 0</pose>
+        <always_on>1</always_on>
+        <update_rate>${fan_rate}</update_rate>
+        <topic>/model/auv/sonar_fan</topic>
+        <gz_frame_id>sonar_fan_link</gz_frame_id>
+        <lidar>
+          <scan>
+            <horizontal>
+              <samples>${fan_samples}</samples>
+              <resolution>1</resolution>
+              <min_angle>-1.48353</min_angle>
+              <max_angle>1.48353</max_angle>
+            </horizontal>
+            <vertical>
+              <samples>1</samples>
+              <resolution>1</resolution>
+              <min_angle>0</min_angle>
+              <max_angle>0</max_angle>
+            </vertical>
+          </scan>
+          <range>
+            <min>0.5</min>
+            <max>100</max>
+            <resolution>0.01</resolution>
+          </range>
+          <noise>
+            <type>gaussian</type>
+            <mean>0</mean>
+            <stddev>0.01</stddev>
+          </noise>
+        </lidar>
+      </sensor>
+      <!--
         DVL beams: 3 x 3 rays looking down, +-30 deg in both directions. The DVL
         node takes the four Janus beams (middle of each edge) for bottom lock and
